File: CANInterfacePCB.kicad_sch (KiCad schematic)
At the start: 0 parts

Commit message: layout sum1 trace
Parts:
- added J1: CH1_in, UTSVT_Connectors:Molex_Nano-Fit_105309-xx02_1x02_P2.50mm_Vertical, symbol utsvt_connectors:CarCANConnector
- added J10: CH1_Debug, UTSVT_Connectors:Molex_Nano-Fit_105309-xx02_1x02_P2.50mm_Vertical, symbol utsvt_connectors:CarCANConnector
- added J11: CH2_Debug, UTSVT_Connectors:Molex_Nano-Fit_105309-xx02_1x02_P2.50mm_Vertical, symbol utsvt_connectors:CarCANConnector
- added J2: CH1_out, UTSVT_Connectors:Molex_Nano-Fit_105309-xx02_1x02_P2.50mm_Vertical, symbol utsvt_connectors:CarCANConnector
- added J3: CH2_in, UTSVT_Connectors:Molex_Nano-Fit_105309-xx02_1x02_P2.50mm_Vertical, symbol utsvt_connectors:CarCANConnector
- added J4: CH2_out, UTSVT_Connectors:Molex_Nano-Fit_105309-xx02_1x02_P2.50mm_Vertical, symbol utsvt_connectors:CarCANConnector
- added J5: CH1_EWERT, footprints:AMPHENOL_L77SDE09SA4CH3R, symbol Connector:DE9_Socket
- added J6: CH2_EWERT, footprints:AMPHENOL_L77SDE09SA4CH3R, symbol Connector:DE9_Socket
- added J7: CH1_PEAK, footprints:AMPHENOL_L77SDE09SA4CH3R, symbol Connector:DE9_Socket
- added J8: CH2_PEAK, footprints:AMPHENOL_L77SDE09SA4CH3R, symbol Connector:DE9_Socket
- added J9: CH1_CH2_Vector, footprints:AMPHENOL_L77SDE09SA4CH3R, symbol Connector:DE9_Socket
- added JP1: CH1_Term, Connector_PinHeader_2.54mm:PinHeader_1x02_P2.54mm_Vertical, symbol Jumper:Jumper_2_Open
- added JP2: CH2_Term, Connector_PinHeader_2.54mm:PinHeader_1x02_P2.54mm_Vertical, symbol Jumper:Jumper_2_Open
- added R1, R2: 120, Resistor_SMD:R_0603_1608Metric, symbol Device:R
Connections:
- new net: JP1.1 (A), R1.2
- new net: JP2.1 (A), R2.2
- new net CH1_CANH: J1.1 (CAN_H), J10.1 (CAN_H), J2.1 (CAN_H), J5.3, J7.7, J9.7, R1.1
- new net CH1_CANL: J1.2 (CAN_L), J10.2 (CAN_L), J2.2 (CAN_L), J5.5, J7.2, J9.2, JP1.2 (B)
- new net CH2_CANH: J11.1 (CAN_H), J3.1 (CAN_H), J4.1 (CAN_H), J6.3, J8.7, J9.8, R2.1
- new net CH2_CANL: J11.2 (CAN_L), J3.2 (CAN_L), J4.2 (CAN_L), J6.5, J8.2, J9.1, JP2.2 (B)
- no-connect marks 0 -> 33
Other:
- note added: "Ewert Candapter"
- note added: "Peak PCAN-USB"
- note added: "Vector VN1610"
