File: CANInterfacePCB.kicad_pcb (KiCad board)
At the start: 2 copper layers, 70.9 x 56.9 mm, 15 parts, among them J1 CH1_in, J10 CH1_Debug, J11 CH2_Debug, J2 CH1_out, J3 CH2_in, J4 CH2_out, J5 CH1_EWERT, J6 CH2_EWERT, J7 CH1_PEAK, J8 CH2_PEAK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

Commit message: Parthiv sucks
Parts:
- moved J4 14.6 mm to (168.4, 55.5)
- moved J3 12.7 mm to (168.6, 70.2), turned to 180 degrees
- moved R2 10.1 mm to (175.4, 55.0), turned to 0 degrees
- moved J2 5.61 mm to (141.1, 64.9), turned to 90 degrees
- moved J5 5.21 mm to (139.4, 46.7)
- moved J7 4.69 mm to (139.0, 84.9)
- moved J1 3.85 mm to (141.2, 55.0), turned to 90 degrees
- moved JP1 3.13 mm to (153.7, 55.0), turned to -90 degrees
- moved R1 3.10 mm to (153.9, 60.2)
- moved JP2 2.91 mm to (182.7, 58.2), turned to -90 degrees
- moved J10 2.68 mm to (152.6, 67.3), turned to 180 degrees
- moved J11 1.90 mm to (180.4, 68.0), turned to 90 degrees
Routing:
- net /CH1_CANH: track 94.0 -> 77.7 mm, vias 0 -> 1
- net /CH2_CANH: track 111.2 -> 102.2 mm
- net /CH1_CANL: track 75.1 -> 67.3 mm
- net Net-(JP2-A): track 5.04 -> 9.65 mm, vias 0 -> 2
- net /CH2_CANL: track 103.3 -> 101.2 mm
- net Net-(JP1-A): track 5.02 -> 4.46 mm
