File: CANInterfacePCB.kicad_pcb (KiCad board)
At the start: 2 copper layers, 70.9 x 56.9 mm, 15 parts, among them J1 CH1_in, J10 CH1_Debug, J11 CH2_Debug, J2 CH1_out, J3 CH2_in, J4 CH2_out, J5 CH1_EWERT, J6 CH2_EWERT, J7 CH1_PEAK, J8 CH2_PEAK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

Commit message: silkscreen
Parts:
- added G***: LOGO, footprints:db9_diagram, B.Cu at (157.3, 65.7)
Routing:
- net /CH1_CANH: track 94.0 -> 86.5 mm, vias 0 -> 1
- net /CH1_CANL: track 75.1 -> 78.9 mm
- net /CH2_CANL: track 103.3 -> 101.5 mm, vias 2 -> 0
- net /CH2_CANH: track 111.2 -> 111.8 mm
Other:
- board text added: "Ewert Candapter: High=3, Low=5 Peak PCAN-USB: High=7, Low=2 Vector VN1610: High_CH1=7, Low_CH1=2 | High_CH2=8, Low_CH2=1"

Commit message: done
Parts:
- added G***: LOGO, LOGO, F.Cu at (161.0, 65.7)
Other:
- board text added: "CH1_debug"
- board text added: "CH2_debug"
